Commit message: review archi for modular end effector

File: ws/src/prl_franka_description/urdf/end_effectors/ball/ball.urdf.xacro (robot description, xacro)
@@ -6,5 +6,5 @@
                 <origin xyz="0 0 0" rpy="0 0 0"/>
                 <geometry>
-                    <mesh filename="file://$(find prl_franka_description)/meshes/end_effectors/ball/ball.stl" scale="0.001 0.001 0.001"/>
+                    <mesh filename="package://prl_franka_description/meshes/end_effectors/ball/ball.stl" scale="0.001 0.001 0.001"/>
                 </geometry>
                 <material name="black">
@@ -15,5 +15,5 @@
                 <origin xyz="0 0 0" rpy="0 0 0"/>
                 <geometry>
-                    <mesh filename="file://$(find prl_franka_description)/meshes/end_effectors/ball/ball_hull.stl" scale="0.001 0.001 0.001"/>
+                    <mesh filename="package://prl_franka_description/meshes/end_effectors/ball/ball_hull.stl" scale="0.001 0.001 0.001"/>
                 </geometry>
             </collision>

File: ws/src/prl_franka_description/urdf/prl_franka.urdf.xacro (robot description, xacro)
@@ -57,5 +57,5 @@
       <visual>
           <geometry>
-              <mesh filename="file://$(find prl_franka_description)/meshes/table.stl" scale="0.001 0.001 0.001"/>
+              <mesh filename="package://prl_franka_description/meshes/table.stl" scale="0.001 0.001 0.001"/>
           </geometry>
           <material name="Blue"/>
@@ -63,5 +63,5 @@
       <collision>
           <geometry>
-              <mesh filename="file://$(find prl_franka_description)/meshes/table.stl" scale="0.001 0.001 0.001"/>
+              <mesh filename="package://prl_franka_description/meshes/table.stl" scale="0.001 0.001 0.001"/>
           </geometry>
       </collision>

Commit message: add ft_sensor

File: ws/src/prl_franka_description/urdf/end_effectors/ball/ball.urdf.xacro (robot description, xacro)
@@ -1,8 +1,8 @@
 <?xml version='1.0' encoding='utf-8'?>
 <robot xmlns:xacro="http://www.ros.org/wiki/xacro" name="ball_effector">
-    <xacro:macro name="ball_effector" params="parent arm_prefix xyz_ee rpy_ee tcp_xyz tcp_rpy">
-        <link name="${arm_prefix}_ball_link">
+    <xacro:macro name="ball_effector" params="parent prefix xyz_ee rpy_ee tcp_xyz tcp_rpy">
+        <link name="${prefix}_ball_link">
             <visual>
-                <origin xyz="0 0 0" rpy="0 0 0"/>
+                <origin xyz="0 0 0.01" rpy="0 0 0"/>
                 <geometry>
                     <mesh filename="package://prl_franka_description/meshes/end_effectors/ball/ball.stl" scale="0.001 0.001 0.001"/>
@@ -23,7 +23,7 @@
             </inertial>
         </link>
-        <joint name="${arm_prefix}_ball_joint" type="fixed">
+        <joint name="${prefix}_ball_joint" type="fixed">
             <parent link="${parent}"/>
-            <child link="${arm_prefix}_ball_link"/>
+            <child link="${prefix}_ball_link"/>
             <origin xyz="${xyz_ee}" rpy="${rpy_ee}"/>
         </joint>

File: ws/src/prl_franka_description/urdf/prl_franka.urdf.xacro (robot description, xacro)
@@ -13,10 +13,9 @@
   <xacro:property name="xyz_ee" value="${' '.join(map(str, ee_pose['xyz']))}"/>
   <xacro:property name="rpy_ee" value="${' '.join(map(str, ee_pose['rpy']))}"/>
+  <xacro:property name="ft_sensor" value="${setup['ROBOT']['force_torque_sensor']}"/>
   <!-- Multi-arm setup? -->
   <xacro:arg name="multi_arm" default="false" />
   <!-- Don't print a prefix for joints, visuals, and links? -->
   <xacro:arg name="no_prefix" default="false"/>
-  <!-- Where is the end-effector connected to, if different from the robot flange?  -->
-  <xacro:arg name="special_connection" default="" />
   <!-- Position offset between ee frame and tcp frame -->
   <xacro:arg name="tcp_xyz" default="0 0 0.1034" />
@@ -43,4 +42,6 @@
   <xacro:arg name="ee_id" default="${ee_id}"/>
   <xacro:arg name="with_sc" default="${with_sc}"/>
+  <xacro:arg name="xyz_ee" default="${xyz_ee}"/>
+  <xacro:arg name="rpy_ee" default="${rpy_ee}"/>
   <!-- Include table-->
   <link name="base_link" />
@@ -80,4 +81,18 @@
     <origin xyz="-0.6 0 0.095" rpy="0 0 0"/>
   </joint>
+  <!-- Force torque sensor -->
+  <xacro:if value="${ft_sensor}">
+    <xacro:include filename="$(find robotiq_ft_sensor_description)/urdf/robotiq_ft300.urdf.xacro" />
+    <xacro:include filename="$(find robotiq_ft_sensor_description)/urdf/robotiq_fts.ros2_control.xacro" />
+      <xacro:robotiq_ft300 parent="${modified_prefix}${arm_id}_link8" tf_prefix="${modified_prefix}">
+        <origin xyz="0 0 -0.01" rpy="0 0 0"/>
+      </xacro:robotiq_ft300>
+    <xacro:property name="ee_mount_parent" value="${modified_prefix}robotiq_ft_frame_id"/>
+  </xacro:if>
+  <xacro:unless value="${ft_sensor}">
+    <xacro:property name="ee_mount_parent" value="${modified_prefix}${arm_id}_link8"/>
+  </xacro:unless>
+  <!-- Where is the end-effector connected to, if different from the robot flange?  -->
+  <xacro:arg name="special_connection" default="${ee_mount_parent}"/>
   <xacro:if value="${ee_id == 'ball' and load_gripper}">
     <xacro:include filename="$(find prl_franka_description)/urdf/end_effectors/ball/ball.urdf.xacro"/>
@@ -104,6 +119,6 @@
         rpy="0 0 0"/>
     <xacro:ball_effector
-        parent="${modified_prefix}${arm_id}_link8"
-        arm_prefix="${modified_prefix}${arm_id}"
+        parent="${ee_mount_parent}"
+        prefix="${modified_prefix}${arm_id}"
         xyz_ee="${xyz_ee}"
         rpy_ee="${rpy_ee}"

Commit message: fix visual and collision frame placements in xacro and add end eff frame at the tip of the sphere

File: ws/src/prl_franka_description/urdf/end_effectors/ball/ball.urdf.xacro (robot description, xacro)
@@ -4,5 +4,5 @@
         <link name="${prefix}_ball_link">
             <visual>
-                <origin xyz="0 0 0.01" rpy="0 0 0"/>
+                <origin xyz="0 0 0.016" rpy="0 0 0"/>
                 <geometry>
                     <mesh filename="package://prl_franka_description/meshes/end_effectors/ball/ball.stl" scale="0.001 0.001 0.001"/>
@@ -13,7 +13,7 @@
             </visual>
             <collision>
-                <origin xyz="0 0 0" rpy="0 0 0"/>
+                <origin xyz="0 0 0.016" rpy="0 0 0"/>
                 <geometry>
-                    <mesh filename="package://prl_franka_description/meshes/end_effectors/ball/ball_hull.stl" scale="0.001 0.001 0.001"/>
+                    <sphere radius="0.02"/>
                 </geometry>
             </collision>
@@ -28,4 +28,10 @@
             <origin xyz="${xyz_ee}" rpy="${rpy_ee}"/>
         </joint>
+        <link name="${prefix}_ee_frame"/>
+        <joint name="${prefix}_ee_joint" type="fixed">
+            <parent link="${prefix}_ball_link"/>
+            <child link="${prefix}_ee_frame"/>
+            <origin xyz="0 0 0.036" rpy="0 0 0"/>
+        </joint>
     </xacro:macro>
 </robot>

File: ws/src/prl_franka_description/urdf/prl_franka.urdf (robot description, URDF)
Before this commit: robot fr3, 16 links, 15 joints
Links:
- added link fr3_ee_frame
- link fr3_ball_link: geometry collision sphere radius=0.02; visual mesh filename=package://prl_franka_description/meshes/end_effectors/ball/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 scale=0.001 0.001 0.001
- link table_link: geometry collision box size=1.0 1.0 0.1; visual mesh filename=package://prl_franka_description/meshes/table.stl scale=0.001 0.001 0.001
Joints:
- added joint fr3_ee_joint: type fixed, parent fr3_ball_link, child fr3_ee_frame, origin xyz=0 0 0.036 rpy=0 0 0
- joint fr3_ball_joint: origin xyz=0.0 0.0 0.0 rpy=0.0 0.0 -2.3561 -> xyz=0.0 0.0 0.0 rpy=0.0 0.0 0.0

File: ws/src/prl_franka_description/urdf/prl_franka.urdf.xacro (robot description, xacro)
@@ -51,6 +51,6 @@
     <origin xyz="0 0 0.68" rpy="0 0 0"/>
   </joint>
-  <material name="Blue">
-    <color rgba="${0/255} ${30/255} ${70/255} 1.0"/>
+  <material name="Beige">
+    <color rgba="${194/255} ${160/255} ${131/255} 1.0"/>
   </material>
   <xacro:arg name="table_scale" default="1 1 1"/>
@@ -60,9 +60,9 @@
               <mesh filename="package://prl_franka_description/meshes/table.stl" scale="0.001 0.001 0.001"/>
           </geometry>
-          <material name="Blue"/>
+          <material name="Beige"/>
       </visual>
       <collision>
           <geometry>
-              <mesh filename="package://prl_franka_description/meshes/table.stl" scale="0.001 0.001 0.001"/>
+              <box size="1.0 1.0 0.1"/>
           </geometry>
       </collision>

Commit message: update ft mount

File: ws/src/prl_franka_description/urdf/end_effectors/ball/ball.urdf.xacro (robot description, xacro)
@@ -4,5 +4,5 @@
         <link name="${prefix}_ball_link">
             <visual>
-                <origin xyz="0 0 0.01" rpy="0 0 0"/>
+                <origin xyz="0 0 0.016" rpy="0 0 0"/>
                 <geometry>
                     <mesh filename="package://prl_franka_description/meshes/end_effectors/ball/ball.stl" scale="0.001 0.001 0.001"/>
@@ -13,5 +13,5 @@
             </visual>
             <collision>
-                <origin xyz="0 0 0" rpy="0 0 0"/>
+                <origin xyz="0 0 0.016" rpy="0 0 0"/>
                 <geometry>
                     <mesh filename="package://prl_franka_description/meshes/end_effectors/ball/ball_hull.stl" scale="0.001 0.001 0.001"/>

File: ws/src/prl_franka_description/urdf/prl_franka.urdf.xacro (robot description, xacro)
@@ -57,4 +57,5 @@
   <link name="table_link">
       <visual>
+          <origin xyz="0 0 -0.05" rpy="0 0 0"/>
           <geometry>
               <mesh filename="package://prl_franka_description/meshes/table.stl" scale="0.001 0.001 0.001"/>
@@ -63,4 +64,5 @@
       </visual>
       <collision>
+          <origin xyz="0 0 -0.05" rpy="0 0 0"/>
           <geometry>
               <mesh filename="package://prl_franka_description/meshes/table.stl" scale="0.001 0.001 0.001"/>
@@ -69,5 +71,5 @@
       <inertial>
           <mass value="10.0"/>
-          <origin xyz="0 0 0" rpy="0 0 0"/>
+          <origin xyz="0 0 -0.050" rpy="0 0 0"/>
           <inertia ixx="1" ixy="0" ixz="0" iyy="1" iyz="0" izz="1"/>
       </inertial>
@@ -79,5 +81,5 @@
     <parent link="table_link"/>
     <child link="${arm_id}_attachment_link"/>
-    <origin xyz="-0.6 0 0.095" rpy="0 0 0"/>
+    <origin xyz="-0.6 0 0.045" rpy="0 0 0"/>
   </joint>
   <!-- Force torque sensor -->
@@ -86,5 +88,5 @@
     <xacro:include filename="$(find robotiq_ft_sensor_description)/urdf/robotiq_fts.ros2_control.xacro" />
       <xacro:robotiq_ft300 parent="${modified_prefix}${arm_id}_link8" tf_prefix="${modified_prefix}">
-        <origin xyz="0 0 -0.01" rpy="0 0 -3.1415"/>
+        <origin xyz="0 0 -0.004" rpy="0 0 -3.1415"/>
       </xacro:robotiq_ft300>
       <!-- args -->
