Commit message: moveit support and ball end effector intagration

File: ws/src/prl_franka_description/urdf/prl_franka.urdf.xacro (robot description, xacro)
@@ -2,21 +2,21 @@
 <robot xmlns:xacro="http://www.ros.org/wiki/xacro" name="fr3">
   <xacro:include filename="$(find franka_description)/robots/common/franka_robot.xacro"/>
-  <xacro:arg name="arm_id" default="fr3" />
-  <!-- The prefix of the robot -->
-  <xacro:arg name="arm_prefix" default="" />
+  <xacro:property name="setup" value="${xacro.load_yaml('$(find prl_franka_run)/config/robot_config.yaml')}"/>
+  <xacro:property name="arm_id" value="${setup['ROBOT']['arm_id']}"/>
+  <xacro:property name="robot_ip" value="${setup['ROBOT']['robot_ip']}"/>
+  <xacro:property name="prefix" value="${setup['ROBOT']['arm_prefix']}"/>
+  <xacro:property name="load_gripper" value="${setup['ROBOT']['load_gripper']}"/>
+  <xacro:property name="ee_id" value="${setup['ROBOT']['ee_id']}"/>
+  <xacro:property name="hand" value="${setup['ROBOT']['load_gripper']}"/>
+  <xacro:property name="with_sc" value="${setup['ROBOT']['self_collision_safety']}"/>
+  <xacro:property name="ee_pose" value="${setup['ROBOT']['end_effector_pose']}"/>
+  <xacro:property name="xyz_ee" value="${' '.join(map(str, ee_pose['xyz']))}"/>
+  <xacro:property name="rpy_ee" value="${' '.join(map(str, ee_pose['rpy']))}"/>
   <!-- Multi-arm setup? -->
   <xacro:arg name="multi_arm" default="false" />
   <!-- Don't print a prefix for joints, visuals, and links? -->
   <xacro:arg name="no_prefix" default="false"/>
-  <!-- Should an end-effector be mounted at the flange?" -->
-  <xacro:arg name="hand" default="true" />
-  <!-- Which end-effector would be mounted at the flange?" -->
-  <xacro:arg name="ee_id" default="franka_hand" />
   <!-- Where is the end-effector connected to, if different from the robot flange?  -->
   <xacro:arg name="special_connection" default="" />
-  <!-- Position offset between ee and parent frame -->
-  <xacro:arg name="xyz_ee" default="0 0 0" />
-  <!-- Rotation offset between ee and parent frame -->
-  <xacro:arg name="rpy_ee" default= "0 0 ${-pi/4}" />
   <!-- Position offset between ee frame and tcp frame -->
   <xacro:arg name="tcp_xyz" default="0 0 0.1034" />
@@ -25,10 +25,6 @@
   <!-- Safety distance for the collision capsules -->
   <xacro:arg name="safety_distance" default="0.03" />
-  <!-- Should self-collision be enabled? -->
-  <xacro:arg name="with_sc" default="false" />
   <!-- Is the robot being controlled with ros2_control?" -->
   <xacro:arg name="ros2_control" default="false" />
-  <!-- IP address or hostname of the robot" -->
-  <xacro:arg name="robot_ip" default="" />
   <!-- Should a fake hardware be used? -->
   <xacro:arg name="use_fake_hardware" default="false" />
@@ -42,6 +38,9 @@
   <xacro:arg name="description_pkg" default="franka_description" />
   <!-- Append an underscore to the user-provided prefix, if non-empty. -->
-  <xacro:property name="prefix" value="$(arg arm_prefix)"/>
   <xacro:property name="modified_prefix" value="${prefix + '_' if prefix else ''}"/>
+  <!-- Copy in arg because franka robot uses this arg in sub macro-->
+  <xacro:arg name="hand" default="${hand}"/>
+  <xacro:arg name="ee_id" default="${ee_id}"/>
+  <xacro:arg name="with_sc" default="${with_sc}"/>
   <!-- Include table-->
   <link name="base_link" />
@@ -74,23 +73,23 @@
   </link>
   <xacro:if value="$(arg gazebo)">
-    <link name="$(arg arm_id)_attachment_link"/>
+    <link name="${arm_id}_attachment_link"/>
   </xacro:if>
-  <joint name="$(arg arm_id)_attachment_joint" type="fixed">
+  <joint name="${arm_id}_attachment_joint" type="fixed">
     <parent link="table_link"/>
-    <child link="$(arg arm_id)_attachment_link"/>
+    <child link="${arm_id}_attachment_link"/>
     <origin xyz="-0.6 0 0.095" rpy="0 0 0"/>
   </joint>
-  <xacro:if value="${'$(arg ee_id)' == 'franka_hand'}">
-    <xacro:franka_robot arm_id="$(arg arm_id)"
-                        joint_limits="${xacro.load_yaml('$(find franka_description)/robots/$(arg arm_id)/joint_limits.yaml')}"
-                        inertials="${xacro.load_yaml('$(find franka_description)/robots/$(arg arm_id)/inertials.yaml')}"
-                        kinematics="${xacro.load_yaml('$(find franka_description)/robots/$(arg arm_id)/kinematics.yaml')}"
-                        dynamics="${xacro.load_yaml('$(find franka_description)/robots/$(arg arm_id)/dynamics.yaml')}"
+  <xacro:if value="${ee_id == 'franka_hand'}">
+    <xacro:franka_robot arm_id="${arm_id}"
+                        joint_limits="${xacro.load_yaml('$(find franka_description)/robots/' + arm_id + '/joint_limits.yaml')}"
+                        inertials="${xacro.load_yaml('$(find franka_description)/robots/' + arm_id + '/inertials.yaml')}"
+                        kinematics="${xacro.load_yaml('$(find franka_description)/robots/' + arm_id + '/kinematics.yaml')}"
+                        dynamics="${xacro.load_yaml('$(find franka_description)/robots/' + arm_id + '/dynamics.yaml')}"
                         gazebo="$(arg gazebo)"
-                        hand="$(arg hand)"
-                        ee_id="$(arg ee_id)"
-                        with_sc="$(arg with_sc)"
+                        hand="${hand}"
+                        ee_id="${ee_id}"
+                        with_sc="${with_sc}"
                         ros2_control="$(arg ros2_control)"
-                        robot_ip="$(arg robot_ip)"
+                        robot_ip="${robot_ip}"
                         use_fake_hardware="$(arg use_fake_hardware)"
                         fake_sensor_commands="$(arg fake_sensor_commands)"
@@ -98,23 +97,23 @@
                         no_prefix="$(arg no_prefix)"
                         arm_prefix="${modified_prefix}"
-                        parent="$(arg arm_id)_attachment_link"
-                        connected_to="$(arg arm_id)_attachment_link"
+                        parent="${arm_id}_attachment_link"
+                        connected_to="${arm_id}_attachment_link"
                         xyz="0 0 0"
                         rpy="0 0 0">
     </xacro:franka_robot>
   </xacro:if>
-  <xacro:if value="${'$(arg ee_id)' == 'ball'}">
+  <xacro:if value="${ee_id == 'ball'}">
     <xacro:include filename="$(find prl_franka_description)/urdf/end_effectors/ball/ball.urdf.xacro"/>
-    <xacro:franka_robot arm_id="$(arg arm_id)"
-                        joint_limits="${xacro.load_yaml('$(find franka_description)/robots/$(arg arm_id)/joint_limits.yaml')}"
-                        inertials="${xacro.load_yaml('$(find franka_description)/robots/$(arg arm_id)/inertials.yaml')}"
-                        kinematics="${xacro.load_yaml('$(find franka_description)/robots/$(arg arm_id)/kinematics.yaml')}"
-                        dynamics="${xacro.load_yaml('$(find franka_description)/robots/$(arg arm_id)/dynamics.yaml')}"
+    <xacro:franka_robot arm_id="${arm_id}"
+                        joint_limits="${xacro.load_yaml('$(find franka_description)/robots/' + arm_id + '/joint_limits.yaml')}"
+                        inertials="${xacro.load_yaml('$(find franka_description)/robots/' + arm_id + '/inertials.yaml')}"
+                        kinematics="${xacro.load_yaml('$(find franka_description)/robots/' + arm_id + '/kinematics.yaml')}"
+                        dynamics="${xacro.load_yaml('$(find franka_description)/robots/' + arm_id + '/dynamics.yaml')}"
                         gazebo="$(arg gazebo)"
                         hand="false"
-                        ee_id=""
-                        with_sc="$(arg with_sc)"
+                        ee_id="none"
+                        with_sc="${with_sc}"
                         ros2_control="$(arg ros2_control)"
-                        robot_ip="$(arg robot_ip)"
+                        robot_ip="${robot_ip}"
                         use_fake_hardware="$(arg use_fake_hardware)"
                         fake_sensor_commands="$(arg fake_sensor_commands)"
@@ -122,10 +121,10 @@
                         no_prefix="$(arg no_prefix)"
                         arm_prefix="${modified_prefix}"
-                        parent="$(arg arm_id)_attachment_link"
-                        connected_to="$(arg arm_id)_attachment_link"
+                        parent="${arm_id}_attachment_link"
+                        connected_to="${arm_id}_attachment_link"
                         xyz="0 0 0"
                         rpy="0 0 0">
     </xacro:franka_robot>
-    <xacro:ball_effector parent="${modified_prefix}$(arg arm_id)_link8" arm_prefix="${modified_prefix}_$(arg arm_id)" xyz_ee="$(arg xyz_ee)" rpy_ee="$(arg rpy_ee)" tcp_xyz="$(arg tcp_xyz)" tcp_rpy="$(arg tcp_rpy)"/>
+    <xacro:ball_effector parent="${modified_prefix}${arm_id}_link8" arm_prefix="${modified_prefix}${arm_id}" xyz_ee="${xyz_ee}" rpy_ee="${rpy_ee}" tcp_xyz="$(arg tcp_xyz)" tcp_rpy="$(arg tcp_rpy)"/>
   </xacro:if>
 </robot>

Commit message: ft_sensor moveit integration and add tare at launch

File: ws/src/prl_franka_description/urdf/prl_franka.urdf.xacro (robot description, xacro)
@@ -6,7 +6,7 @@
   <xacro:property name="robot_ip" value="${setup['ROBOT']['robot_ip']}"/>
   <xacro:property name="prefix" value="${setup['ROBOT']['arm_prefix']}"/>
-  <xacro:property name="load_gripper" value="${setup['ROBOT']['load_gripper']}"/>
+  <xacro:property name="load_end_effector" value="${setup['ROBOT']['load_end_effector']}"/>
   <xacro:property name="ee_id" value="${setup['ROBOT']['ee_id']}"/>
-  <xacro:property name="hand" value="${setup['ROBOT']['load_gripper']}"/>
+  <xacro:property name="hand" value="${setup['ROBOT']['load_end_effector']}"/>
   <xacro:property name="with_sc" value="${setup['ROBOT']['self_collision_safety']}"/>
   <xacro:property name="ee_pose" value="${setup['ROBOT']['end_effector_pose']}"/>
@@ -108,5 +108,5 @@
   <!-- Where is the end-effector connected to, if different from the robot flange?  -->
   <xacro:arg name="special_connection" default="${ee_mount_parent}"/>
-  <xacro:if value="${ee_id == 'ball' and load_gripper}">
+  <xacro:if value="${ee_id == 'ball' and load_end_effector}">
     <xacro:include filename="$(find prl_franka_description)/urdf/end_effectors/ball/ball.urdf.xacro"/>
     <xacro:franka_robot

Commit message: update frame placement

File: ws/src/prl_franka_description/urdf/prl_franka.urdf.xacro (robot description, xacro)
@@ -86,5 +86,5 @@
     <xacro:include filename="$(find robotiq_ft_sensor_description)/urdf/robotiq_fts.ros2_control.xacro" />
       <xacro:robotiq_ft300 parent="${modified_prefix}${arm_id}_link8" tf_prefix="${modified_prefix}">
-        <origin xyz="0 0 -0.01" rpy="0 0 0"/>
+        <origin xyz="0 0 -0.01" rpy="0 0 -3.1415"/>
       </xacro:robotiq_ft300>
       <!-- args -->

Commit message: Update prl_franka.urdf.xacro

File: ws/src/prl_franka_description/urdf/prl_franka.urdf.xacro (robot description, xacro)
@@ -64,7 +64,7 @@
       </visual>
       <collision>
-          <origin xyz="0 0 -0.05" rpy="0 0 0"/>
+          <origin xyz="0 0 -0.365" rpy="0 0 0"/>
           <geometry>
-              <box size="1.0 1.0 0.1"/>
+              <box size="1.0 1.0 0.73"/>
           </geometry>
       </collision>

Commit message: fix ft sensor

File: ws/src/prl_franka_description/urdf/prl_franka.urdf.xacro (robot description, xacro)
@@ -38,4 +38,5 @@
   <!-- Append an underscore to the user-provided prefix, if non-empty. -->
   <xacro:property name="modified_prefix" value="${prefix + '_' if prefix else ''}"/>
+  <xacro:arg name="use_ft_sensor" default="false"/>
   <!-- Copy in arg because franka robot uses this arg in sub macro-->
   <xacro:arg name="hand" default="${hand}"/>
@@ -86,14 +87,15 @@
   <xacro:if value="${ft_sensor}">
     <xacro:include filename="$(find robotiq_ft_sensor_description)/urdf/robotiq_ft300.urdf.xacro" />
-    <xacro:include filename="$(find robotiq_ft_sensor_description)/urdf/robotiq_fts.ros2_control.xacro" />
-      <xacro:robotiq_ft300 parent="${modified_prefix}${arm_id}_link8" tf_prefix="${modified_prefix}">
-        <origin xyz="0 0 -0.004" rpy="0 0 -3.1415"/>
-      </xacro:robotiq_ft300>
-      <!-- args -->
-      <xacro:arg name="use_fake_mode" default="false"/>
-      <xacro:arg name="max_retries" default="100"/>
-      <xacro:arg name="read_rate" default="100"/>
-      <xacro:arg name="ftdi_id" default=""/>
-      <!-- robotiq sensor hardware -->
+    <xacro:robotiq_ft300 parent="${modified_prefix}${arm_id}_link8" prefix="${modified_prefix}">
+      <origin xyz="0 0 -0.004" rpy="0 0 0"/>
+    </xacro:robotiq_ft300>
+    <!-- args -->
+    <xacro:arg name="use_fake_mode" default="false"/>
+    <xacro:arg name="max_retries" default="100"/>
+    <xacro:arg name="read_rate" default="100"/>
+    <xacro:arg name="ftdi_id" default=""/>
+    <!-- robotiq sensor hardware -->
+    <xacro:if value="$(arg ros2_control)">
+      <xacro:include filename="$(find robotiq_ft_sensor_description)/urdf/robotiq_fts.ros2_control.xacro" />
       <xacro:robotiq_fts_ros2_control
           tf_prefix="${modified_prefix}"
@@ -103,4 +105,5 @@
           ftdi_id="$(arg ftdi_id)"
       />
+    </xacro:if>
     <xacro:property name="ee_mount_parent" value="${modified_prefix}robotiq_ft_frame_id"/>
   </xacro:if>

Commit message: Update prl_franka.urdf.xacro

File: ws/src/prl_franka_description/urdf/prl_franka.urdf.xacro (robot description, xacro)
@@ -88,5 +88,5 @@
     <xacro:include filename="$(find robotiq_ft_sensor_description)/urdf/robotiq_ft300.urdf.xacro" />
     <xacro:robotiq_ft300 parent="${modified_prefix}${arm_id}_link8" prefix="${modified_prefix}">
-      <origin xyz="0 0 -0.004" rpy="0 0 0"/>
+      <origin xyz="0 0 0" rpy="0 0 0"/>
     </xacro:robotiq_ft300>
     <!-- args -->
