Commit message: Fix generated URDF's absolute paths

File: ws/src/prl_franka_description/urdf/prl_franka.urdf (robot description, URDF)
Before this commit: robot fr3, 13 links, 12 joints
Links:
- link fr3_ball_link: geometry collision mesh filename=package://prl_franka_description/meshes/end_effectors/ball/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 scale=0.001 0.001 0.001; visual mesh filename=package://prl_franka_description/meshes/end_effectors/ball/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 scale=0.001 0.001 0.001
- link table_link: geometry collision mesh filename=package://prl_franka_description/meshes/table.stl scale=0.001 0.001 0.001; visual mesh filename=package://prl_franka_description/meshes/table.stl scale=0.001 0.001 0.001

Commit message: change service name

File: ws/src/prl_franka_description/urdf/prl_franka.urdf (robot description, URDF)
Before this commit: robot fr3, 13 links, 12 joints
Links:
- added link ft300_mounting_plate; collision mesh filename=package://robotiq_ft_sensor_description/meshes/collision/mo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; visual mesh filename=package://robotiq_ft_sensor_description/meshes/visual/mount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
- added link ft300_sensor, mass 0.300; collision mesh filename=package://robotiq_ft_sensor_description/meshes/collision/ro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; visual mesh filename=package://robotiq_ft_sensor_description/meshes/visual/robot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
- added link robotiq_ft_frame_id
Joints:
- added joint ft300_fix: type fixed, parent fr3_link8, child ft300_mounting_plate, origin xyz=0 0 -0.01 rpy=0 0 0
- added joint ft300_mounting_plate_joint: type fixed, parent ft300_mounting_plate, child ft300_sensor, origin xyz=0 0 0.0415 rpy=0 3.141592653589793 0
- added joint measurment_joint: type fixed, parent ft300_sensor, child robotiq_ft_frame_id, origin xyz=0 0 0 rpy=0 3.141592653589793 -1.5707963267948966
- joint fr3_ball_joint: origin xyz=0.0 0.0 0.01 rpy=0.0 0.0 0.0 -> xyz=0.0 0.0 0.0 rpy=0.0 0.0 -2.3561; parent fr3_link8 -> robotiq_ft_frame_id

Commit message: Update prl_franka.urdf

File: ws/src/prl_franka_description/urdf/prl_franka.urdf (robot description, URDF)
Before this commit: robot fr3, 16 links, 15 joints
Joints:
- joint ft300_fix: origin xyz=0 0 -0.01 rpy=0 0 0 -> xyz=0 0 -0.01 rpy=0 0 -3.1415

Commit message: generate urdf from xacro

File: ws/src/prl_franka_description/urdf/prl_franka.urdf (robot description, URDF)
Before this commit: robot fr3, 17 links, 16 joints
Links:
- link table_link: geometry collision box size=1.0 1.0 0.73; visual mesh filename=package://prl_franka_description/meshes/table.stl scale=0.001 0.001 0.001
Joints:
- joint fr3_attachment_joint: origin xyz=-0.6 0 0.095 rpy=0 0 0 -> xyz=-0.6 0 0.045 rpy=0 0 0
- joint ft300_fix: origin xyz=0 0 -0.01 rpy=0 0 -3.1415 -> xyz=0 0 0 rpy=0 0 0
