Commit message: fixed config file sensor setup & added tare option

File: prl_franka_description/urdf/prl_franka.urdf.xacro (robot description, xacro)
@@ -13,5 +13,5 @@
   <xacro:property name="xyz_ee" value="${' '.join(map(str, ee_pose['xyz']))}"/>
   <xacro:property name="rpy_ee" value="${' '.join(map(str, ee_pose['rpy']))}"/>
-  <xacro:property name="ft_sensor" value="${setup['ROBOT']['force_torque_sensor']}"/>
+  <xacro:property name="ft_sensor" value="${setup['ROBOT']['use_ft_sensor']}"/>
   <!-- Multi-arm setup? -->
   <xacro:arg name="multi_arm" default="false" />
